Commit message: dataset naprawiony

File: ai_slam_ws/src/ai_slam_description/urdf/diffbot.urdf (robot description, URDF)
Before this commit: robot diffbot, 2 links, 1 joints
Links:
- added link base_footprint
- added link base_inertia, mass 5.0
- added link world
- link base_link: mass 5.0 -> None
Joints:
- added joint base_footprint_joint: type fixed, parent base_footprint, child base_link, origin xyz=0 0 0 rpy=0 0 0
- added joint base_inertia_joint: type fixed, parent base_link, child base_inertia, origin xyz=0 0 0 rpy=0 0 0
- added joint base_joint: type fixed, parent world, child base_footprint, origin xyz=0 0 0 rpy=0 0 0
- joint laser_joint: origin xyz=0.12 0.0 0.15 rpy=0 0 0 -> xyz=0.0 0.0 0.15 rpy=0 0 0

Commit message: Poprawa loggowania danych + pełen config

File: ai_slam_ws/src/ai_slam_description/urdf/diffbot.urdf (robot description, URDF)
Before this commit: robot diffbot, 5 links, 4 joints
Links:
- removed link base_footprint
- removed link world
Joints:
- removed joint base_footprint_joint
- removed joint base_joint

Commit message: dodanie Scan-to-scan

File: ai_slam_ws/src/ai_slam_description/urdf/diffbot.urdf (robot description, URDF)
Before this commit: robot diffbot, 3 links, 2 joints
Links:
- removed link base_inertia
- added link caster_link, mass 0.05; collision sphere radius=0.035; visual sphere radius=0.035
- added link left_wheel_link, mass 0.3; collision cylinder length=0.03 radius=0.035; visual cylinder length=0.03 radius=0.035
- added link right_wheel_link, mass 0.3; collision cylinder length=0.03 radius=0.035; visual cylinder length=0.03 radius=0.035
- link base_link: mass None -> 5.0; geometry collision box size=0.30 0.20 0.10; visual box size=0.30 0.20 0.10
- link laser_link: geometry collision cylinder length=0.05 radius=0.035; visual cylinder length=0.05 radius=0.035
Joints:
- removed joint base_inertia_joint
- added joint caster_joint: type fixed, parent base_link, child caster_link, origin xyz=0.115 0 0 rpy=0 0 0
- added joint left_wheel_joint: type revolute, parent base_link, child left_wheel_link, origin xyz=-0.12 0.105 0 rpy=1.5708 0 0, axis 0 1 0, limit lower=-1e16 upper=1e16 effort=0 velocity=0
- added joint right_wheel_joint: type revolute, parent base_link, child right_wheel_link, origin xyz=-0.12 -0.105 0 rpy=1.5708 0 0, axis 0 1 0, limit lower=-1e16 upper=1e16 effort=0 velocity=0
- joint laser_joint: origin xyz=0.0 0.0 0.15 rpy=0 0 0 -> xyz=-0.05 0 0.15 rpy=0 0 0

Commit message: sweep

File: ai_slam_ws/src/ai_slam_description/urdf/diffbot.urdf (robot description, URDF)
Before this commit: robot diffbot, 5 links, 4 joints
Links:
- added link base_link_inertia, mass 5.0
- link base_link: mass 5.0 -> None
Joints:
- added joint base_link_inertia_joint: type fixed, parent base_link, child base_link_inertia, origin xyz=0 0 0 rpy=0 0 0
